Commit message: Updated measurements according to data sheet.

File: ROS/catkin_workspace/src/minibot/urdf/minibot.urdf (robot description, URDF)
Before this commit: robot minibot, 5 links, 4 joints
Links:
- link base_link: geometry visual box size=0.19 0.13 0.06

Commit message: Added real measurements of base, laser and IMU.

File: ROS/catkin_workspace/src/minibot/urdf/minibot.urdf (robot description, URDF)
Before this commit: robot minibot, 5 links, 4 joints
Links:
- link base_link: geometry visual box size=0.17 0.126 0.051

Commit message: Fixed base and wheel size.

File: ROS/catkin_workspace/src/minibot/urdf/minibot.urdf (robot description, URDF)
Before this commit: robot minibot, 5 links, 4 joints
Links:
- link base_link: geometry visual box size=0.17 0.079 0.051
- link wheel_1: geometry visual cylinder length=0.0235 radius=0.025
- link wheel_2: geometry visual cylinder length=0.0235 radius=0.025
- link wheel_3: geometry visual cylinder length=0.0235 radius=0.025
- link wheel_4: geometry visual cylinder length=0.0235 radius=0.025

Commit message: Added collision and inertial.

File: ROS/catkin_workspace/src/minibot/urdf/minibot.urdf (robot description, URDF)
Before this commit: robot minibot, 5 links, 4 joints
Links:
- link base_link: mass None -> 10; geometry collision box size=0.17 0.079 0.051; visual box size=0.17 0.079 0.051
- link wheel_1: mass None -> 10; geometry collision cylinder length=0.0235 radius=0.025; visual cylinder length=0.0235 radius=0.025
- link wheel_2: mass None -> 10; geometry collision cylinder length=0.0235 radius=0.025; visual cylinder length=0.0235 radius=0.025
- link wheel_3: mass None -> 10; geometry collision cylinder length=0.0235 radius=0.025; visual cylinder length=0.0235 radius=0.025
- link wheel_4: mass None -> 10; geometry collision cylinder length=0.0235 radius=0.025; visual cylinder length=0.0235 radius=0.025
