Commit message: Updated materials

File: ROS/catkin_workspace/src/minibot/urdf/minibot.urdf.xacro (robot description, xacro)
@@ -8,4 +8,14 @@
   <xacro:property name="wheeldiam" value="0.07" />
   <xacro:property name="pi" value="3.1415" />
+  <!-- Materials -->
+  <material name="silver">
+    <color rgba="0.75 0.75 0.75 1"/>
+  </material>
+  <material name="blue">
+    <color rgba="0 0 0.8 1"/>
+  </material>
+  <material name="black">
+    <color rgba="0 0 0 1"/>
+  </material>
   <material name="white">
     <color rgba="1 1 1 1"/>
@@ -13,16 +23,4 @@
 </robot>
 - - - old URDF:
-<?xml version="1.0"?>
-<robot name="minibot">
-  <!-- Materials -->
-  <material name="silver">
-    <color rgba="0.75 0.75 0.75 1"/>
-  </material>
-  <material name="blue">
-      <color rgba="0 0 0.8 1"/>
-    </material>
-    <material name="black">
-      <color rgba="0 0 0 1"/>
-    </material>
   <!--
   The chassis.
@@ -157,3 +155,2 @@
     <origin xyz="0 0 0"/>
   </joint>
-</robot>

Commit message: Added inertial

File: ROS/catkin_workspace/src/minibot/urdf/minibot.urdf.xacro (robot description, xacro)
@@ -21,4 +21,11 @@
     <color rgba="1 1 1 1"/>
   </material>
+  <!-- Inertial -->
+  <xacro:macro name="default_inertial" params="mass">
+    <inertial>
+      <mass value="${mass}" />
+      <inertia ixx="0.1" ixy="0.0" ixz="0.0" iyy="0.1" iyz="0.0" izz="0.1"/>
+    </inertial>
+  </xacro:macro>
 </robot>
 - - - old URDF:

Commit message: Completed new base_link with xacro.

File: ROS/catkin_workspace/src/minibot/urdf/minibot.urdf.xacro (robot description, xacro)
@@ -1,5 +1,8 @@
 <?xml version="1.0"?>
 <robot xmlns:xacro="http://www.ros.org/wiki/xacro" name="minibot">
-  <xacro:property name="width" value="0.2" />
+  <!-- chassis -->
+  <xacro:property name="length" value="0.17" />
+  <xacro:property name="width" value="0.079" />
+  <xacro:property name="height" value="0.051" />
   <xacro:property name="leglen" value="0.6" />
   <xacro:property name="polelen" value="0.2" />
@@ -29,30 +32,39 @@
   </xacro:macro>
 </robot>
+<!--
+The chassis.
+"base_link" is a more common name for a chassis in ROS.
+-->
+<link name="base_link">
+  <visual>
+    <geometry>
+      <box size="${length} ${width} ${height}"/>
+    </geometry>
+    <!-- ORIGIN OF THE BASE?!?     <origin rpy="0 0 0" xyz="0 0 0.03"/> -->
+    <material name="silver"/>
+  </visual>
+  <collision>
+    <geometry>
+      <box size="${length} ${width} ${height}"/>
+    </geometry>
+  </collision>
+  <xacro:default_inertial mass="1"/>
+</link>
 - - - old URDF:
-  <!--
-  The chassis.
-  "base_link" is a more common name for a chassis in ROS.
-  -->
+  <!-- Wheel 1 -->
   <link name="base_link">
     <visual>
       <geometry>
-        <!-- A rectangle, sized in meters. Measured on the Arexx RP5. -->
-        <!-- The grey box, without wheels for visualisation reasons. -->
-        <box size="0.17 0.079 0.051"/>
+        <cylinder radius="${width}" length="${bodylen}"/>
       </geometry>
-      <!-- ORIGIN OF THE BASE?!?     <origin rpy="0 0 0" xyz="0 0 0.03"/> -->
-    <material name="silver"/>
+      <material name="blue"/>
     </visual>
     <collision>
-       <geometry>
-         <box size="0.17 0.079 0.051"/>
-       </geometry>
-     </collision>
-     <inertial>
-       <mass value="10"/>
-       <inertia ixx="0.1" ixy="0.0" ixz="0.0" iyy="0.1" iyz="0.0" izz="0.1"/>
-     </inertial>
-</link>
-  <!-- Wheel 1 -->
+      <geometry>
+        <cylinder radius="${width}" length="${bodylen}"/>
+      </geometry>
+    </collision>
+    <xacro:default_inertial mass="10"/>
+  </link>
   <link name="wheel_1">
     <visual>

Commit message: Added constants, updated comments.

File: ROS/catkin_workspace/src/minibot/urdf/minibot.urdf.xacro (robot description, xacro)
@@ -5,5 +5,7 @@
   <xacro:property name="width" value="0.079" />
   <xacro:property name="height" value="0.051" />
-  <xacro:property name="leglen" value="0.6" />
+  <!-- wheel depth is 2.35 cm overall with rubber -->
+  <xacro:property name="wheellength" value="0.0235" />
+  <xacro:property name="wheelradius" value="0.025" />
   <xacro:property name="polelen" value="0.2" />
   <xacro:property name="bodylen" value="0.6" />
@@ -24,5 +26,5 @@
     <color rgba="1 1 1 1"/>
   </material>
-  <!-- Inertial -->
+  <!-- Default Inertial -->
   <xacro:macro name="default_inertial" params="mass">
     <inertial>

Commit message: Moved wheel code up, to be updated.

File: ROS/catkin_workspace/src/minibot/urdf/minibot.urdf.xacro (robot description, xacro)
@@ -53,46 +53,46 @@
   <xacro:default_inertial mass="1"/>
 </link>
+<!-- Wheel 1 -->
+<link name="base_link">
+  <visual>
+    <geometry>
+      <cylinder radius="${width}" length="${bodylen}"/>
+    </geometry>
+    <material name="blue"/>
+  </visual>
+  <collision>
+    <geometry>
+      <cylinder radius="${width}" length="${bodylen}"/>
+    </geometry>
+  </collision>
+  <xacro:default_inertial mass="1"/>
+</link>
+<link name="wheel_1">
+  <visual>
+    <geometry>
+      <!-- wheel depth is 2.35 cm overall with rubber -->
+      <cylinder length="0.0235" radius="0.025"/>
+    </geometry>
+    <!--
+    origin roll,pitch,yaw and x,y,z
+    1. We rotate the wheel by PI/2 (~1.5) around the Y axis (pitch)
+    2. We move the origin +5.65 cm (11.3 cm/2) to the front (+x)
+       and +3.95 cm (7.9cm/2) to the left of the center (+y)
+       and -0.65 cm (3cm - 2,35cm) down from the center (-z).
+    -->
+    <origin rpy="0 1.5 1.5" xyz="0.0565 0.0395 -0.0065"/>
+    <material name="black"/>
+  </visual>
+  <collision>
+     <geometry>
+       <cylinder length="0.0235" radius="0.025"/>
+     </geometry>
+   </collision>
+   <inertial>
+     <mass value="10"/>
+     <inertia ixx="0.1" ixy="0.0" ixz="0.0" iyy="0.1" iyz="0.0" izz="0.1"/>
+   </inertial>
+</link>
 - - - old URDF:
-  <!-- Wheel 1 -->
-  <link name="base_link">
-    <visual>
-      <geometry>
-        <cylinder radius="${width}" length="${bodylen}"/>
-      </geometry>
-      <material name="blue"/>
-    </visual>
-    <collision>
-      <geometry>
-        <cylinder radius="${width}" length="${bodylen}"/>
-      </geometry>
-    </collision>
-    <xacro:default_inertial mass="10"/>
-  </link>
-  <link name="wheel_1">
-    <visual>
-      <geometry>
-        <!-- wheel depth is 2.35 cm overall with rubber -->
-        <cylinder length="0.0235" radius="0.025"/>
-      </geometry>
-      <!--
-      origin roll,pitch,yaw and x,y,z
-      1. We rotate the wheel by PI/2 (~1.5) around the Y axis (pitch)
-      2. We move the origin +5.65 cm (11.3 cm/2) to the front (+x)
-         and +3.95 cm (7.9cm/2) to the left of the center (+y)
-         and -0.65 cm (3cm - 2,35cm) down from the center (-z).
-      -->
-      <origin rpy="0 1.5 1.5" xyz="0.0565 0.0395 -0.0065"/>
-      <material name="black"/>
-    </visual>
-    <collision>
-       <geometry>
-         <cylinder length="0.0235" radius="0.025"/>
-       </geometry>
-     </collision>
-     <inertial>
-       <mass value="10"/>
-       <inertia ixx="0.1" ixy="0.0" ixz="0.0" iyy="0.1" iyz="0.0" izz="0.1"/>
-     </inertial>
-  </link>
   <!-- Wheel 2 -->
   <link name="wheel_2">

Commit message: Fixed copy error

File: ROS/catkin_workspace/src/minibot/urdf/minibot.urdf.xacro (robot description, xacro)
@@ -54,18 +54,4 @@
 </link>
 <!-- Wheel 1 -->
-<link name="base_link">
-  <visual>
-    <geometry>
-      <cylinder radius="${width}" length="${bodylen}"/>
-    </geometry>
-    <material name="blue"/>
-  </visual>
-  <collision>
-    <geometry>
-      <cylinder radius="${width}" length="${bodylen}"/>
-    </geometry>
-  </collision>
-  <xacro:default_inertial mass="1"/>
-</link>
 <link name="wheel_1">
   <visual>

Commit message: Replaced wheel measurements and inertial by xacro macro.

File: ROS/catkin_workspace/src/minibot/urdf/minibot.urdf.xacro (robot description, xacro)
@@ -57,6 +57,5 @@
   <visual>
     <geometry>
-      <!-- wheel depth is 2.35 cm overall with rubber -->
-      <cylinder length="0.0235" radius="0.025"/>
+      <cylinder length="${wheellength}" radius="${wheelradius}"/>
     </geometry>
     <!--
@@ -72,11 +71,8 @@
   <collision>
      <geometry>
-       <cylinder length="0.0235" radius="0.025"/>
+       <cylinder length="${wheellength}" radius="${wheelradius}"/>
      </geometry>
    </collision>
-   <inertial>
-     <mass value="10"/>
-     <inertia ixx="0.1" ixy="0.0" ixz="0.0" iyy="0.1" iyz="0.0" izz="0.1"/>
-   </inertial>
+   <xacro:default_inertial mass="1"/>
 </link>
 - - - old URDF:

Commit message: Same for wheel 2

File: ROS/catkin_workspace/src/minibot/urdf/minibot.urdf.xacro (robot description, xacro)
@@ -76,24 +76,21 @@
    <xacro:default_inertial mass="1"/>
 </link>
+<!-- Wheel 2 -->
+<link name="wheel_2">
+  <visual>
+    <geometry>
+      <cylinder length="${wheellength}" radius="${wheelradius}"/>
+    </geometry>
+    <origin rpy="0 1.5 1.5" xyz="-0.0565 0.0395 -0.0065"/>
+    <material name="black"/>
+  </visual>
+  <collision>
+     <geometry>
+       <cylinder length="${wheellength}" radius="${wheelradius}"/>
+     </geometry>
+   </collision>
+   <xacro:default_inertial mass="1"/>
+</link>
 - - - old URDF:
-  <!-- Wheel 2 -->
-  <link name="wheel_2">
-    <visual>
-      <geometry>
-        <cylinder length="0.0235" radius="0.025"/>
-      </geometry>
-      <origin rpy="0 1.5 1.5" xyz="-0.0565 0.0395 -0.0065"/>
-      <material name="black"/>
-    </visual>
-    <collision>
-       <geometry>
-         <cylinder length="0.0235" radius="0.025"/>
-       </geometry>
-     </collision>
-     <inertial>
-       <mass value="10"/>
-       <inertia ixx="0.1" ixy="0.0" ixz="0.0" iyy="0.1" iyz="0.0" izz="0.1"/>
-     </inertial>
-  </link>
   <!-- Wheel 3 -->
   <link name="wheel_3">

Commit message: Same for wheel 3 and 4

File: ROS/catkin_workspace/src/minibot/urdf/minibot.urdf.xacro (robot description, xacro)
@@ -92,43 +92,37 @@
    <xacro:default_inertial mass="1"/>
 </link>
+<!-- Wheel 3 -->
+<link name="wheel_3">
+  <visual>
+    <geometry>
+      <cylinder length="${wheellength}" radius="${wheelradius}"/>
+    </geometry>
+    <origin rpy="0 1.5 1.5" xyz="0.0565 -0.0395 -0.0065"/>
+    <material name="black"/>
+  </visual>
+  <collision>
+     <geometry>
+       <cylinder length="${wheellength}" radius="${wheelradius}"/>
+     </geometry>
+   </collision>
+   <xacro:default_inertial mass="1"/>
+</link>
+<!-- Wheel 4 -->
+<link name="wheel_4">
+  <visual>
+    <geometry>
+      <cylinder length="${wheellength}" radius="${wheelradius}"/>
+    </geometry>
+    <origin rpy="0 1.5 1.5" xyz="-0.0565 -0.0395 -0.0065"/>
+    <material name="black"/>
+  </visual>
+  <collision>
+     <geometry>
+       <cylinder length="${wheellength}" radius="${wheelradius}"/>
+     </geometry>
+   </collision>
+   <xacro:default_inertial mass="1"/>
+</link>
 - - - old URDF:
-  <!-- Wheel 3 -->
-  <link name="wheel_3">
-    <visual>
-      <geometry>
-        <cylinder length="0.0235" radius="0.025"/>
-      </geometry>
-      <origin rpy="0 1.5 1.5" xyz="0.0565 -0.0395 -0.0065"/>
-      <material name="black"/>
-    </visual>
-    <collision>
-       <geometry>
-         <cylinder length="0.0235" radius="0.025"/>
-       </geometry>
-     </collision>
-     <inertial>
-       <mass value="10"/>
-       <inertia ixx="0.1" ixy="0.0" ixz="0.0" iyy="0.1" iyz="0.0" izz="0.1"/>
-     </inertial>
-  </link>
-  <!-- Wheel 4 -->
-  <link name="wheel_4">
-    <visual>
-      <geometry>
-        <cylinder length="0.0235" radius="0.025"/>
-      </geometry>
-      <origin rpy="0 1.5 1.5" xyz="-0.0565 -0.0395 -0.0065"/>
-      <material name="black"/>
-    </visual>
-    <collision>
-       <geometry>
-         <cylinder length="0.0235" radius="0.025"/>
-       </geometry>
-     </collision>
-     <inertial>
-       <mass value="10"/>
-       <inertia ixx="0.1" ixy="0.0" ixz="0.0" iyy="0.1" iyz="0.0" izz="0.1"/>
-     </inertial>
-  </link>
   <!-- Joint for wheel 1 -->
   <joint name="base_to_wheel1" type="continuous">

Commit message: removed duplicate tag, updated indentions.

File: ROS/catkin_workspace/src/minibot/urdf/minibot.urdf.xacro (robot description, xacro)
@@ -33,36 +33,35 @@
     </inertial>
   </xacro:macro>
-</robot>
-<!--
-The chassis.
-"base_link" is a more common name for a chassis in ROS.
--->
-<link name="base_link">
-  <visual>
-    <geometry>
-      <box size="${length} ${width} ${height}"/>
-    </geometry>
-    <!-- ORIGIN OF THE BASE?!?     <origin rpy="0 0 0" xyz="0 0 0.03"/> -->
-    <material name="silver"/>
-  </visual>
-  <collision>
-    <geometry>
-      <box size="${length} ${width} ${height}"/>
-    </geometry>
-  </collision>
-  <xacro:default_inertial mass="1"/>
-</link>
-<!-- Wheel 1 -->
-<link name="wheel_1">
-  <visual>
-    <geometry>
-      <cylinder length="${wheellength}" radius="${wheelradius}"/>
-    </geometry>
-    <!--
-    origin roll,pitch,yaw and x,y,z
-    1. We rotate the wheel by PI/2 (~1.5) around the Y axis (pitch)
-    2. We move the origin +5.65 cm (11.3 cm/2) to the front (+x)
-       and +3.95 cm (7.9cm/2) to the left of the center (+y)
-       and -0.65 cm (3cm - 2,35cm) down from the center (-z).
+  <!--
+  The chassis.
+  "base_link" is a more common name for a chassis in ROS.
+  -->
+  <link name="base_link">
+    <visual>
+      <geometry>
+        <box size="${length} ${width} ${height}"/>
+      </geometry>
+      <!-- ORIGIN OF THE BASE?!?     <origin rpy="0 0 0" xyz="0 0 0.03"/> -->
+      <material name="silver"/>
+    </visual>
+    <collision>
+      <geometry>
+        <box size="${length} ${width} ${height}"/>
+      </geometry>
+    </collision>
+    <xacro:default_inertial mass="1"/>
+  </link>
+  <!-- Wheel 1 -->
+  <link name="wheel_1">
+    <visual>
+      <geometry>
+        <cylinder length="${wheellength}" radius="${wheelradius}"/>
+      </geometry>
+      <!--
+      origin roll,pitch,yaw and x,y,z
+      1. We rotate the wheel by PI/2 (~1.5) around the Y axis (pitch)
+      2. We move the origin +5.65 cm (11.3 cm/2) to the front (+x)
+      and +3.95 cm (7.9cm/2) to the left of the center (+y)
+      and -0.65 cm (3cm - 2,35cm) down from the center (-z).
     -->
     <origin rpy="0 1.5 1.5" xyz="0.0565 0.0395 -0.0065"/>
@@ -70,58 +69,58 @@
   </visual>
   <collision>
-     <geometry>
-       <cylinder length="${wheellength}" radius="${wheelradius}"/>
-     </geometry>
-   </collision>
-   <xacro:default_inertial mass="1"/>
-</link>
-<!-- Wheel 2 -->
-<link name="wheel_2">
-  <visual>
     <geometry>
       <cylinder length="${wheellength}" radius="${wheelradius}"/>
     </geometry>
-    <origin rpy="0 1.5 1.5" xyz="-0.0565 0.0395 -0.0065"/>
-    <material name="black"/>
-  </visual>
-  <collision>
-     <geometry>
-       <cylinder length="${wheellength}" radius="${wheelradius}"/>
-     </geometry>
-   </collision>
-   <xacro:default_inertial mass="1"/>
-</link>
-<!-- Wheel 3 -->
-<link name="wheel_3">
-  <visual>
-    <geometry>
-      <cylinder length="${wheellength}" radius="${wheelradius}"/>
-    </geometry>
-    <origin rpy="0 1.5 1.5" xyz="0.0565 -0.0395 -0.0065"/>
-    <material name="black"/>
-  </visual>
-  <collision>
-     <geometry>
-       <cylinder length="${wheellength}" radius="${wheelradius}"/>
-     </geometry>
-   </collision>
-   <xacro:default_inertial mass="1"/>
-</link>
-<!-- Wheel 4 -->
-<link name="wheel_4">
-  <visual>
-    <geometry>
-      <cylinder length="${wheellength}" radius="${wheelradius}"/>
-    </geometry>
-    <origin rpy="0 1.5 1.5" xyz="-0.0565 -0.0395 -0.0065"/>
-    <material name="black"/>
-  </visual>
-  <collision>
-     <geometry>
-       <cylinder length="${wheellength}" radius="${wheelradius}"/>
-     </geometry>
-   </collision>
-   <xacro:default_inertial mass="1"/>
-</link>
+  </collision>
+  <xacro:default_inertial mass="1"/>
+  </link>
+  <!-- Wheel 2 -->
+  <link name="wheel_2">
+    <visual>
+      <geometry>
+        <cylinder length="${wheellength}" radius="${wheelradius}"/>
+      </geometry>
+      <origin rpy="0 1.5 1.5" xyz="-0.0565 0.0395 -0.0065"/>
+      <material name="black"/>
+    </visual>
+    <collision>
+      <geometry>
+        <cylinder length="${wheellength}" radius="${wheelradius}"/>
+      </geometry>
+    </collision>
+    <xacro:default_inertial mass="1"/>
+  </link>
+  <!-- Wheel 3 -->
+  <link name="wheel_3">
+    <visual>
+      <geometry>
+        <cylinder length="${wheellength}" radius="${wheelradius}"/>
+      </geometry>
+      <origin rpy="0 1.5 1.5" xyz="0.0565 -0.0395 -0.0065"/>
+      <material name="black"/>
+    </visual>
+    <collision>
+      <geometry>
+        <cylinder length="${wheellength}" radius="${wheelradius}"/>
+      </geometry>
+    </collision>
+    <xacro:default_inertial mass="1"/>
+  </link>
+  <!-- Wheel 4 -->
+  <link name="wheel_4">
+    <visual>
+      <geometry>
+        <cylinder length="${wheellength}" radius="${wheelradius}"/>
+      </geometry>
+      <origin rpy="0 1.5 1.5" xyz="-0.0565 -0.0395 -0.0065"/>
+      <material name="black"/>
+    </visual>
+    <collision>
+      <geometry>
+        <cylinder length="${wheellength}" radius="${wheelradius}"/>
+      </geometry>
+    </collision>
+    <xacro:default_inertial mass="1"/>
+  </link>
   <!-- Joint for wheel 1 -->
   <joint name="base_to_wheel1" type="continuous">

Commit message: Replaced values with constants and some math now

File: ROS/catkin_workspace/src/minibot/urdf/minibot.urdf.xacro (robot description, xacro)
@@ -8,8 +8,5 @@
   <xacro:property name="wheellength" value="0.0235" />
   <xacro:property name="wheelradius" value="0.025" />
-  <xacro:property name="polelen" value="0.2" />
-  <xacro:property name="bodylen" value="0.6" />
-  <xacro:property name="baselen" value="0.4" />
-  <xacro:property name="wheeldiam" value="0.07" />
+  <!-- constant pi -->
   <xacro:property name="pi" value="3.1415" />
   <!-- Materials -->
@@ -60,10 +57,10 @@
       <!--
       origin roll,pitch,yaw and x,y,z
-      1. We rotate the wheel by PI/2 (~1.5) around the Y axis (pitch)
+      1. We rotate the wheel by PI/2 around the Y axis (pitch)
       2. We move the origin +5.65 cm (11.3 cm/2) to the front (+x)
       and +3.95 cm (7.9cm/2) to the left of the center (+y)
       and -0.65 cm (3cm - 2,35cm) down from the center (-z).
     -->
-    <origin rpy="0 1.5 1.5" xyz="0.0565 0.0395 -0.0065"/>
+    <origin rpy="0 ${pi/2} ${pi/2}" xyz="0.0565 0.0395 -0.0065"/>
     <material name="black"/>
   </visual>
@@ -81,5 +78,5 @@
         <cylinder length="${wheellength}" radius="${wheelradius}"/>
       </geometry>
-      <origin rpy="0 1.5 1.5" xyz="-0.0565 0.0395 -0.0065"/>
+      <origin rpy="0 ${pi/2} ${pi/2}" xyz="-0.0565 0.0395 -0.0065"/>
       <material name="black"/>
     </visual>
@@ -97,5 +94,5 @@
         <cylinder length="${wheellength}" radius="${wheelradius}"/>
       </geometry>
-      <origin rpy="0 1.5 1.5" xyz="0.0565 -0.0395 -0.0065"/>
+      <origin rpy="0 ${pi/2} ${pi/2}" xyz="0.0565 -0.0395 -0.0065"/>
       <material name="black"/>
     </visual>
@@ -113,5 +110,5 @@
         <cylinder length="${wheellength}" radius="${wheelradius}"/>
       </geometry>
-      <origin rpy="0 1.5 1.5" xyz="-0.0565 -0.0395 -0.0065"/>
+      <origin rpy="0 ${pi/2} ${pi/2}" xyz="-0.0565 -0.0395 -0.0065"/>
       <material name="black"/>
     </visual>

Commit message: removed pi due to new global definement

File: ROS/catkin_workspace/src/minibot/urdf/minibot.urdf.xacro (robot description, xacro)
@@ -8,6 +8,4 @@
   <xacro:property name="wheellength" value="0.0235" />
   <xacro:property name="wheelradius" value="0.025" />
-  <!-- constant pi -->
-  <xacro:property name="pi" value="3.1415" />
   <!-- Materials -->
   <material name="silver">

Commit message: Changed wheel joints back to fixed

File: ROS/catkin_workspace/src/minibot/urdf/minibot.urdf.xacro (robot description, xacro)
@@ -119,5 +119,5 @@
   </link>
   <!-- Joint for wheel 1 -->
-  <joint name="base_to_wheel1" type="continuous">
+  <joint name="base_to_wheel1" type="fixed">
     <parent link="base_link"/>
     <child link="wheel_1"/>
@@ -125,5 +125,5 @@
   </joint>
   <!-- Joint for wheel 2 -->
-  <joint name="base_to_wheel2" type="continuous">
+  <joint name="base_to_wheel2" type="fixed">
     <parent link="base_link"/>
     <child link="wheel_2"/>
@@ -131,5 +131,5 @@
   </joint>
   <!-- Joint for wheel 3 -->
-  <joint name="base_to_wheel3" type="continuous">
+  <joint name="base_to_wheel3" type="fixed">
     <parent link="base_link"/>
     <child link="wheel_3"/>
@@ -137,5 +137,5 @@
   </joint>
   <!-- Joint for wheel 4 -->
-  <joint name="base_to_wheel4" type="continuous">
+  <joint name="base_to_wheel4" type="fixed">
     <parent link="base_link"/>
     <child link="wheel_4"/>

Commit message: Fixed indention

File: ROS/catkin_workspace/src/minibot/urdf/minibot.urdf.xacro (robot description, xacro)
@@ -3,5 +3,5 @@
   <!-- chassis -->
   <xacro:property name="length" value="0.17" />
-  <xacro:property name="width" value="0.079" />
+  <xacro:property name="width"  value="0.079" />
   <xacro:property name="height" value="0.051" />
   <!-- wheel depth is 2.35 cm overall with rubber -->

Commit message: Defined some components (laser, PCB, RasPi...)

File: ROS/catkin_workspace/src/minibot/urdf/minibot.urdf.xacro (robot description, xacro)
@@ -5,4 +5,23 @@
   <xacro:property name="width"  value="0.079" />
   <xacro:property name="height" value="0.051" />
+  <!-- main PCB board on top -->
+  <xacro:property name="PCBlength" value="0.17" />
+  <xacro:property name="PCBwidth"  value="0.126" />
+  <xacro:property name="PCBheight" value="0.004" />
+  <!-- IMU board BNO055 (mounted) -->
+  <xacro:property name="IMUlength" value="0.020" />
+  <xacro:property name="IMUwidth"  value="0.027" />
+  <xacro:property name="IMUheight" value="0.010" />
+  <!-- Raspberry Pi (mounted) -->
+  <xacro:property name="IMUlength" value="0.085" />
+  <xacro:property name="IMUwidth"  value="0.056" />
+  <xacro:property name="IMUheight" value="0.030" />
+  <!-- Hokuyo laser rangefinder - base -->
+  <xacro:property name="laserLength" value="0.05" />
+  <xacro:property name="laserWidth"  value="0.05" />
+  <xacro:property name="laserHeight" value="0.041" />
+  <!-- Hokuyo laser rangefinder - cylinder -->
+  <xacro:property name="laserCylLength" value="0.0265" />
+  <xacro:property name="laserCylRadius" value="0.0375" />
   <!-- wheel depth is 2.35 cm overall with rubber -->
   <xacro:property name="wheellength" value="0.0235" />
@@ -20,4 +39,8 @@
   <material name="white">
     <color rgba="1 1 1 1"/>
+  </material>
+  <!-- #B9 A7 76 = 185 167 118 -->
+  <material name="euroPCB">
+    <color rgba="0.73 0.65 0.46 1"/>
   </material>
   <!-- Default Inertial -->
