Commit message: Added main PCB and IMU to visuals

File: ROS/catkin_workspace/src/minibot/urdf/minibot.urdf.xacro (robot description, xacro)
@@ -70,4 +70,38 @@
     <xacro:default_inertial mass="1"/>
   </link>
+  <!-- the main PCB on top of the chassis, where everything is mounted -->
+  <link name="mainPCB">
+    <visual>
+      <geometry>
+        <box size="${PCBlength} ${PCBwidth} ${PCBheight}"/>
+      </geometry>
+      <!-- Located on top of the base -->
+      <origin rpy="0 0 0" xyz="0 0 -${height/2}"/>
+      <material name="euroPCB"/>
+    </visual>
+    <collision>
+      <geometry>
+        <box size="${PCBlength} ${PCBwidth} ${PCBheight}"/>
+      </geometry>
+    </collision>
+    <xacro:default_inertial mass="1"/>
+  </link>
+  <!-- the IMU on the main PCB -->
+  <link name="IMU">
+    <visual>
+      <geometry>
+        <box size="${IMUlength} ${IMUwidth} ${IMUheight}"/>
+      </geometry>
+      <!-- Located on top of the base, on top of the PCB -->
+      <origin rpy="0 0 0" xyz="0 0 -${(height/2)+PCBwidth}"/>
+      <material name="Blue"/>
+    </visual>
+    <collision>
+      <geometry>
+        <box size="${IMUlength} ${IMUwidth} ${IMUheight}"/>
+      </geometry>
+    </collision>
+    <xacro:default_inertial mass="1"/>
+  </link>
   <!-- Wheel 1 -->
   <link name="wheel_1">

Commit message: Added missing joints for mainPCB and IMU

File: ROS/catkin_workspace/src/minibot/urdf/minibot.urdf.xacro (robot description, xacro)
@@ -199,3 +199,15 @@
     <origin xyz="0 0 0"/>
   </joint>
+  <!-- Joint for mainPCB -->
+  <joint name="base_to_mainPCB" type="fixed">
+    <parent link="base_link"/>
+    <child link="mainPCB"/>
+    <origin xyz="0 0 0"/>
+  </joint>
+  <!-- Joint for IMU -->
+  <joint name="base_to_IMU" type="fixed">
+    <parent link="base_link"/>
+    <child link="IMU"/>
+    <origin xyz="0 0 0"/>
+  </joint>
 </robot>

Commit message: Fixed IMU and mainPCB positions

File: ROS/catkin_workspace/src/minibot/urdf/minibot.urdf.xacro (robot description, xacro)
@@ -79,5 +79,5 @@
       </geometry>
       <!-- Located on top of the base -->
-      <origin rpy="0 0 0" xyz="0 0 -${height/2}"/>
+      <origin rpy="0 0 0" xyz="0 0 ${height/2}"/>
       <material name="euroPCB"/>
     </visual>
@@ -96,5 +96,5 @@
       </geometry>
       <!-- Located on top of the base, on top of the PCB -->
-      <origin rpy="0 0 0" xyz="0 0 -${(height/2)+PCBwidth}"/>
+      <origin rpy="0 0 0" xyz="0 0 ${(height/2)+PCBheight}"/>
       <material name="Blue"/>
     </visual>

Commit message: Fixed paste errors.

File: ROS/catkin_workspace/src/minibot/urdf/minibot.urdf.xacro (robot description, xacro)
@@ -16,7 +16,7 @@
   <xacro:property name="IMUheight" value="0.010" />
   <!-- Raspberry Pi (mounted) -->
-  <xacro:property name="IMUlength" value="0.085" />
-  <xacro:property name="IMUwidth"  value="0.056" />
-  <xacro:property name="IMUheight" value="0.030" />
+  <xacro:property name="Raspilength" value="0.085" />
+  <xacro:property name="Raspiwidth"  value="0.056" />
+  <xacro:property name="Raspiheight" value="0.030" />
   <!-- Hokuyo laser rangefinder - base -->
   <xacro:property name="laserLength" value="0.05" />

Commit message: fixed color

File: ROS/catkin_workspace/src/minibot/urdf/minibot.urdf.xacro (robot description, xacro)
@@ -97,5 +97,5 @@
       <!-- Located on top of the base, on top of the PCB -->
       <origin rpy="0 0 0" xyz="0 0 ${(height/2)+PCBheight}"/>
-      <material name="Blue"/>
+      <material name="blue"/>
     </visual>
     <collision>

Commit message: Added laser base visual and joint, updated length name.

File: ROS/catkin_workspace/src/minibot/urdf/minibot.urdf.xacro (robot description, xacro)
@@ -20,7 +20,7 @@
   <xacro:property name="Raspiheight" value="0.030" />
   <!-- Hokuyo laser rangefinder - base -->
-  <xacro:property name="laserLength" value="0.05" />
-  <xacro:property name="laserWidth"  value="0.05" />
-  <xacro:property name="laserHeight" value="0.041" />
+  <xacro:property name="laserBaseLength" value="0.05" />
+  <xacro:property name="laserBaseWidth"  value="0.05" />
+  <xacro:property name="laserBaseHeight" value="0.041" />
   <!-- Hokuyo laser rangefinder - cylinder -->
   <xacro:property name="laserCylLength" value="0.0265" />
@@ -106,4 +106,21 @@
     <xacro:default_inertial mass="1"/>
   </link>
+    <!-- the Laser base on the main PCB -->
+    <link name="laserBase">
+      <visual>
+        <geometry>
+          <box size="${laserBaseLength} ${laserBaseWidth} ${laserBaseHeight}"/>
+        </geometry>
+        <!-- Located on top of the base, on top of the PCB, to the front (x) -->
+        <origin rpy="0 0 0" xyz="${(length/2)-(laserBaseLength/2)} 0 ${(height/2)+PCBheight+(laserBaseHeight/2)}"/>
+        <material name="black"/>
+      </visual>
+      <collision>
+        <geometry>
+          <box size="${laserBaseLength} ${laserBaseWidth} ${laserBaseHeight}"/>
+        </geometry>
+      </collision>
+      <xacro:default_inertial mass="1"/>
+    </link>
   <!-- Wheel 1 -->
   <link name="wheel_1">
@@ -213,3 +230,9 @@
     <origin xyz="0 0 0"/>
   </joint>
+  <!-- Joint for laser base -->
+  <joint name="base_to_laserBase" type="fixed">
+    <parent link="base_link"/>
+    <child link="laserBase"/>
+    <origin xyz="0 0 0"/>
+  </joint>
 </robot>

Commit message: fixed indention

File: ROS/catkin_workspace/src/minibot/urdf/minibot.urdf.xacro (robot description, xacro)
@@ -106,21 +106,21 @@
     <xacro:default_inertial mass="1"/>
   </link>
-    <!-- the Laser base on the main PCB -->
-    <link name="laserBase">
-      <visual>
-        <geometry>
-          <box size="${laserBaseLength} ${laserBaseWidth} ${laserBaseHeight}"/>
-        </geometry>
-        <!-- Located on top of the base, on top of the PCB, to the front (x) -->
-        <origin rpy="0 0 0" xyz="${(length/2)-(laserBaseLength/2)} 0 ${(height/2)+PCBheight+(laserBaseHeight/2)}"/>
-        <material name="black"/>
-      </visual>
-      <collision>
-        <geometry>
-          <box size="${laserBaseLength} ${laserBaseWidth} ${laserBaseHeight}"/>
-        </geometry>
-      </collision>
-      <xacro:default_inertial mass="1"/>
-    </link>
+  <!-- the Laser base on the main PCB -->
+  <link name="laserBase">
+    <visual>
+      <geometry>
+        <box size="${laserBaseLength} ${laserBaseWidth} ${laserBaseHeight}"/>
+      </geometry>
+      <!-- Located on top of the base, on top of the PCB, to the front (x) -->
+      <origin rpy="0 0 0" xyz="${(length/2)-(laserBaseLength/2)} 0 ${(height/2)+PCBheight+(laserBaseHeight/2)}"/>
+      <material name="black"/>
+    </visual>
+    <collision>
+      <geometry>
+        <box size="${laserBaseLength} ${laserBaseWidth} ${laserBaseHeight}"/>
+      </geometry>
+    </collision>
+    <xacro:default_inertial mass="1"/>
+  </link>
   <!-- Wheel 1 -->
   <link name="wheel_1">

Commit message: Fixed laser head radius

File: ROS/catkin_workspace/src/minibot/urdf/minibot.urdf.xacro (robot description, xacro)
@@ -25,5 +25,5 @@
   <!-- Hokuyo laser rangefinder - cylinder -->
   <xacro:property name="laserCylLength" value="0.0265" />
-  <xacro:property name="laserCylRadius" value="0.0375" />
+  <xacro:property name="laserCylRadius" value="0.01875" />
   <!-- wheel depth is 2.35 cm overall with rubber -->
   <xacro:property name="wheellength" value="0.0235" />

Commit message: Added laser head visual and joint

File: ROS/catkin_workspace/src/minibot/urdf/minibot.urdf.xacro (robot description, xacro)
@@ -123,4 +123,21 @@
     <xacro:default_inertial mass="1"/>
   </link>
+    <!-- the Laser "head" (cylinder) on the lase base -->
+    <link name="laserHead">
+      <visual>
+        <geometry>
+          <cylinder length="${laserCylLength}" radius="${laserCylRadius}"/>
+        </geometry>
+        <!-- Located on top of the base, on top of the PCB, on top of the laser base, to the front (x) -->
+        <origin rpy="0 0 0" xyz="${(length/2)-(laserBaseLength/2)} 0 ${(height/2)+PCBheight+laserBaseHeight+(laserCylLength/2)}"/>
+        <material name="black"/>
+      </visual>
+      <collision>
+        <geometry>
+          <cylinder length="${laserCylLength}" radius="${laserCylRadius}"/>
+        </geometry>
+      </collision>
+      <xacro:default_inertial mass="1"/>
+    </link>
   <!-- Wheel 1 -->
   <link name="wheel_1">
@@ -236,3 +253,9 @@
     <origin xyz="0 0 0"/>
   </joint>
+  <!-- Joint for laser "head" (cylinder) -->
+  <joint name="base_to_laserHead" type="fixed">
+    <parent link="base_link"/>
+    <child link="laserHead"/>
+    <origin xyz="0 0 0"/>
+  </joint>
 </robot>
